Commit message: IMU sensor reading in RViz

File: wcr_description/urdf/wcr_base.xacro (robot description, xacro)
@@ -26,4 +26,9 @@
     </joint>
     <link name="imu_link">
+        <inertial>
+            <origin xyz="0 0 0" rpy="0 0 0"/>
+            <mass value="0.05"/>
+            <inertia ixx="1e-5" ixy="0" ixz="0" iyy="1e-5" iyz="0" izz="1e-5"/>
+        </inertial>
     </link>
     <!-- T265 LINK -->
@@ -367,11 +372,3 @@
 		</collision>
 	</link>
-    <gazebo reference="imu_link">
-        <sensor name="imu_sensor" type="imu">
-            <update_rate>100</update_rate>
-            <always_on>true</always_on>
-            <topic>imu</topic>
-            <visualize>true</visualize>
-        </sensor>
-    </gazebo>
 </robot>
